File: CAN-Accessories_Board/CAN_Accessories.sch (KiCad schematic (older format))
At the start: 47 parts, among them J1 39301040, J2 39301040, J3 39301040, J4 39301040, J5 39301040, J6 39301040, J7 39301060, J8 39301060, Q1 Q_NMOS_SGD, Q2 Q_NMOS_SGD, Q3 Q_NMOS_SGD, Q4 Q_NMOS_SGD, Q5 Q_NMOS_SGD, Q6 Q_NMOS_SGD, U1 NUCLEO_L432KC, U2 MCP2562FD-E_SN

Commit message: Changed layout
Parts:
- added R14, R15, R16: 10K, Resistor_SMD:R_0603_1608Metric, symbol Device:R
- U2: footprint SOIC8-N_MC_MCH -> MCP2562FD-E_SN:MCP2562FD-E_SN
Connections:
- wire segments 149 -> 160
Other:
- moved on the sheet: JP1, JP2, JP3
Changed lines of the file:
@@
 L Jumper:SolderJumper_2_Open JP1
 U 1 1 6041A3F4
-P 4900 2500
-F 0 "JP1" H 5350 2500 50  0000 C CNN
-F 1 "SolderJumper_2_Open" H 5850 2500 50  0000 C CNN
-F 2 "Jumper:SolderJumper-2_P1.3mm_Open_Pad1.0x1.5mm" H 4900 2500 50  0001 C CNN
-F 3 "~" H 4900 2500 50  0001 C CNN
-	1    4900 2500
+P 5250 2500
+F 0 "JP1" H 5700 2500 50  0000 C CNN
+F 1 "SolderJumper_2_Open" H 6200 2500 50  0000 C CNN
+F 2 "Jumper:SolderJumper-2_P1.3mm_Open_Pad1.0x1.5mm" H 5250 2500 50  0001 C CNN
+F 3 "~" H 5250 2500 50  0001 C CNN
+	1    5250 2500
 	1    0    0    -1
 $EndComp
@@
 L Jumper:SolderJumper_2_Open JP2
 U 1 1 60432AAF
-P 4900 2600
-F 0 "JP2" H 5350 2600 50  0000 C CNN
-F 1 "SolderJumper_2_Open" H 5850 2600 50  0000 C CNN
-F 2 "Jumper:SolderJumper-2_P1.3mm_Open_Pad1.0x1.5mm" H 4900 2600 50  0001 C CNN
-F 3 "~" H 4900 2600 50  0001 C CNN
-	1    4900 2600
+P 5250 2600
+F 0 "JP2" H 5700 2600 50  0000 C CNN
+F 1 "SolderJumper_2_Open" H 6200 2600 50  0000 C CNN
+F 2 "Jumper:SolderJumper-2_P1.3mm_Open_Pad1.0x1.5mm" H 5250 2600 50  0001 C CNN
+F 3 "~" H 5250 2600 50  0001 C CNN
+	1    5250 2600
 	1    0    0    -1
 $EndComp
@@
 L Jumper:SolderJumper_2_Open JP3
 U 1 1 6043E5F0
-P 4900 2700
-F 0 "JP3" H 5350 2700 50  0000 C CNN
-F 1 "SolderJumper_2_Open" H 5850 2700 50  0000 C CNN
-F 2 "Jumper:SolderJumper-2_P1.3mm_Open_Pad1.0x1.5mm" H 4900 2700 50  0001 C CNN
-F 3 "~" H 4900 2700 50  0001 C CNN
-	1    4900 2700
-	1    0    0    -1
-$EndComp
-Wire Wire Line
-	5150 2700 5050 2700
-Wire Wire Line
-	5050 2600 5150 2600
-Connection ~ 5150 2600
-Wire Wire Line
-	5150 2600 5150 2700
-Wire Wire Line
-	5050 2500 5150 2500
-Wire Wire Line
-	5150 2500 5150 2600
+P 5250 2700
+F 0 "JP3" H 5700 2700 50  0000 C CNN
+F 1 "SolderJumper_2_Open" H 6200 2700 50  0000 C CNN
+F 2 "Jumper:SolderJumper-2_P1.3mm_Open_Pad1.0x1.5mm" H 5250 2700 50  0001 C CNN
+F 3 "~" H 5250 2700 50  0001 C CNN
+	1    5250 2700
+	1    0    0    -1
+$EndComp
+Wire Wire Line
+	5500 2700 5400 2700
+Wire Wire Line
+	5400 2600 5500 2600
+Connection ~ 5500 2600
+Wire Wire Line
+	5500 2600 5500 2700
+Wire Wire Line
+	5400 2500 5500 2500
+Wire Wire Line
+	5500 2500 5500 2600
 Text Label 2900 1600 0    50   ~ 0
 STBY
@@
 	4000 4250 4000 4400
 Wire Wire Line
-	5150 2700 5150 2900
-Connection ~ 5150 2700
+	5500 2700 5500 2900
+Connection ~ 5500 2700
 $Comp
 L power:+12V #PWR0115
@@
 Text Label 4650 1900 0    50   ~ 0
 5V
-Text Label 4850 2900 0    50   ~ 0
+Text Label 5200 2900 0    50   ~ 0
 3V3
 Text Label 7450 1700 0    50   ~ 0
@@
 	3900 6700 3900 6900
 Wire Wire Line
-	4400 2900 5150 2900
-Wire Wire Line
-	4400 2700 4750 2700
-Wire Wire Line
-	4400 2600 4750 2600
-Wire Wire Line
-	4400 2500 4750 2500
+	4400 2900 5500 2900
+Wire Wire Line
+	4400 2700 5000 2700
+Wire Wire Line
+	4400 2500 4500 2500
 Wire Wire Line
 	3300 2200 2900 2200
@@
 F 0 "U2" H 9050 2087 60  0000 C CNN
 F 1 "MCP2562FD-E_SN" H 9050 1981 60  0000 C CNN
-F 2 "SOIC8-N_MC_MCH" H 9050 1940 60  0001 C CNN
+F 2 "MCP2562FD-E_SN:MCP2562FD-E_SN" H 9050 1940 60  0001 C CNN
 F 3 "" H 8250 1700 60  0000 C CNN
 	1    9050 1600
 	1    0    0    -1
 $EndComp
+$Comp
+L Device:R R14
+U 1 1 604D3925
+P 4500 3150
+F 0 "R14" H 4550 3200 50  0000 L CNN
+F 1 "10K" H 4550 3100 50  0000 L CNN
+F 2 "Resistor_SMD:R_0603_1608Metric" V 4430 3150 50  0001 C CNN
+F 3 "~" H 4500 3150 50  0001 C CNN
+	1    4500 3150
+	1    0    0    -1
+$EndComp
+$Comp
+L Device:R R15
+U 1 1 604D4814
+P 4750 3150
+F 0 "R15" H 4800 3200 50  0000 L CNN
+F 1 "10K" H 4800 3100 50  0000 L CNN
+F 2 "Resistor_SMD:R_0603_1608Metric" V 4680 3150 50  0001 C CNN
+F 3 "~" H 4750 3150 50  0001 C CNN
+	1    4750 3150
+	1    0    0    -1
+$EndComp
+$Comp
+L Device:R R16
+U 1 1 604D5327
+P 5000 3150
+F 0 "R16" H 5050 3200 50  0000 L CNN
+F 1 "10K" H 5050 3100 50  0000 L CNN
+F 2 "Resistor_SMD:R_0603_1608Metric" V 4930 3150 50  0001 C CNN
+F 3 "~" H 5000 3150 50  0001 C CNN
+	1    5000 3150
+	1    0    0    -1
+$EndComp
+Wire Wire Line
+	4500 3000 4500 2500
+Connection ~ 4500 2500
+Wire Wire Line
+	4500 2500 5100 2500
+Wire Wire Line
+	4750 3000 4750 2600
+Wire Wire Line
+	4400 2600 4750 2600
+Connection ~ 4750 2600
+Wire Wire Line
+	4750 2600 5100 2600
+Wire Wire Line
+	5000 3000 5000 2700
+Connection ~ 5000 2700
+Wire Wire Line
+	5000 2700 5100 2700
+$Comp
+L power:GND #PWR0102
+U 1 1 60504710
+P 4750 3350
+F 0 "#PWR0102" H 4750 3100 50  0001 C CNN
+F 1 "GND" H 4755 3177 50  0000 C CNN
+F 2 "" H 4750 3350 50  0001 C CNN
+F 3 "" H 4750 3350 50  0001 C CNN
+	1    4750 3350
+	1    0    0    -1
+$EndComp
+Wire Wire Line
+	4500 3300 4500 3350
+Wire Wire Line
+	5000 3350 5000 3300
+Wire Wire Line
+	4500 3350 4750 3350
+Connection ~ 4750 3350
+Wire Wire Line
+	4750 3350 5000 3350
+Wire Wire Line
+	4750 3300 4750 3350
 $EndSCHEMATC

Commit message: Changed footprints from 0603 to 0805
Parts:
- C1, C2: footprint Capacitor_SMD:C_0603_1608Metric -> Capacitor_SMD:C_0805_2012Metric
- D1, D2, D3, D4, D5, D6: footprint LED_SMD:LED_0603_1608Metric -> LED_SMD:LED_0805_2012Metric
- R1, R10, R11, R12, R13, R14, R15, R16, R2, R3, R4, R5, R6, R7, R8, R9: footprint Resistor_SMD:R_0603_1608Metric -> Resistor_SMD:R_0805_2012Metric
Changed lines of the file:
@@
 F 0 "R2" H 1270 6346 50  0000 L CNN
 F 1 "10K" H 1270 6255 50  0000 L CNN
-F 2 "Resistor_SMD:R_0603_1608Metric" V 1130 6300 50  0001 C CNN
+F 2 "Resistor_SMD:R_0805_2012Metric" V 1130 6300 50  0001 C CNN
 F 3 "~" H 1200 6300 50  0001 C CNN
 	1    1200 6300
@@
 F 0 "R4" H 2270 6346 50  0000 L CNN
 F 1 "10K" H 2270 6255 50  0000 L CNN
-F 2 "Resistor_SMD:R_0603_1608Metric" V 2130 6300 50  0001 C CNN
+F 2 "Resistor_SMD:R_0805_2012Metric" V 2130 6300 50  0001 C CNN
 F 3 "~" H 2200 6300 50  0001 C CNN
 	1    2200 6300
@@
 F 0 "R6" H 3270 6346 50  0000 L CNN
 F 1 "10K" H 3270 6255 50  0000 L CNN
-F 2 "Resistor_SMD:R_0603_1608Metric" V 3130 6300 50  0001 C CNN
+F 2 "Resistor_SMD:R_0805_2012Metric" V 3130 6300 50  0001 C CNN
 F 3 "~" H 3200 6300 50  0001 C CNN
 	1    3200 6300
@@
 F 0 "R8" H 4270 6346 50  0000 L CNN
 F 1 "10K" H 4270 6255 50  0000 L CNN
-F 2 "Resistor_SMD:R_0603_1608Metric" V 4130 6300 50  0001 C CNN
+F 2 "Resistor_SMD:R_0805_2012Metric" V 4130 6300 50  0001 C CNN
 F 3 "~" H 4200 6300 50  0001 C CNN
 	1    4200 6300
@@
 F 0 "R10" H 5270 6346 50  0000 L CNN
 F 1 "10K" H 5270 6255 50  0000 L CNN
-F 2 "Resistor_SMD:R_0603_1608Metric" V 5130 6300 50  0001 C CNN
+F 2 "Resistor_SMD:R_0805_2012Metric" V 5130 6300 50  0001 C CNN
 F 3 "~" H 5200 6300 50  0001 C CNN
 	1    5200 6300
@@
 F 0 "R12" H 6270 6346 50  0000 L CNN
 F 1 "10K" H 6270 6255 50  0000 L CNN
-F 2 "Resistor_SMD:R_0603_1608Metric" V 6130 6300 50  0001 C CNN
+F 2 "Resistor_SMD:R_0805_2012Metric" V 6130 6300 50  0001 C CNN
 F 3 "~" H 6200 6300 50  0001 C CNN
 	1    6200 6300
@@
 F 0 "R13" H 8320 3746 50  0000 L CNN
 F 1 "120" H 8320 3655 50  0000 L CNN
-F 2 "Resistor_SMD:R_0603_1608Metric" V 8180 3700 50  0001 C CNN
+F 2 "Resistor_SMD:R_0805_2012Metric" V 8180 3700 50  0001 C CNN
 F 3 "~" H 8250 3700 50  0001 C CNN
 	1    8250 3700
@@
 F 0 "D1" V 939 6282 50  0000 R CNN
 F 1 "LED" V 848 6282 50  0000 R CNN
-F 2 "LED_SMD:LED_0603_1608Metric" H 900 6400 50  0001 C CNN
+F 2 "LED_SMD:LED_0805_2012Metric" H 900 6400 50  0001 C CNN
 F 3 "~" H 900 6400 50  0001 C CNN
 	1    900  6400
@@
 F 0 "D2" V 1939 6282 50  0000 R CNN
 F 1 "LED" V 1848 6282 50  0000 R CNN
-F 2 "LED_SMD:LED_0603_1608Metric" H 1900 6400 50  0001 C CNN
+F 2 "LED_SMD:LED_0805_2012Metric" H 1900 6400 50  0001 C CNN
 F 3 "~" H 1900 6400 50  0001 C CNN
 	1    1900 6400
@@
 F 0 "D3" V 2939 6282 50  0000 R CNN
 F 1 "LED" V 2848 6282 50  0000 R CNN
-F 2 "LED_SMD:LED_0603_1608Metric" H 2900 6400 50  0001 C CNN
+F 2 "LED_SMD:LED_0805_2012Metric" H 2900 6400 50  0001 C CNN
 F 3 "~" H 2900 6400 50  0001 C CNN
 	1    2900 6400
@@
 F 0 "D4" V 3939 6282 50  0000 R CNN
 F 1 "LED" V 3848 6282 50  0000 R CNN
-F 2 "LED_SMD:LED_0603_1608Metric" H 3900 6400 50  0001 C CNN
+F 2 "LED_SMD:LED_0805_2012Metric" H 3900 6400 50  0001 C CNN
 F 3 "~" H 3900 6400 50  0001 C CNN
 	1    3900 6400
@@
 F 0 "D5" V 4939 6282 50  0000 R CNN
 F 1 "LED" V 4848 6282 50  0000 R CNN
-F 2 "LED_SMD:LED_0603_1608Metric" H 4900 6400 50  0001 C CNN
+F 2 "LED_SMD:LED_0805_2012Metric" H 4900 6400 50  0001 C CNN
 F 3 "~" H 4900 6400 50  0001 C CNN
 	1    4900 6400
@@
 F 0 "D6" V 5939 6282 50  0000 R CNN
 F 1 "LED" V 5848 6282 50  0000 R CNN
-F 2 "LED_SMD:LED_0603_1608Metric" H 5900 6400 50  0001 C CNN
+F 2 "LED_SMD:LED_0805_2012Metric" H 5900 6400 50  0001 C CNN
 F 3 "~" H 5900 6400 50  0001 C CNN
 	1    5900 6400
@@
 F 0 "C2" H 10215 2146 50  0000 L CNN
 F 1 "100nF" H 10215 2055 50  0000 L CNN
-F 2 "Capacitor_SMD:C_0603_1608Metric" H 10138 1950 50  0001 C CNN
+F 2 "Capacitor_SMD:C_0805_2012Metric" H 10138 1950 50  0001 C CNN
 F 3 "~" H 10100 2100 50  0001 C CNN
 	1    10100 2100
@@
 F 0 "C1" H 7765 2146 50  0000 L CNN
 F 1 "100nF" H 7765 2055 50  0000 L CNN
-F 2 "Capacitor_SMD:C_0603_1608Metric" H 7688 1950 50  0001 C CNN
+F 2 "Capacitor_SMD:C_0805_2012Metric" H 7688 1950 50  0001 C CNN
 F 3 "~" H 7650 2100 50  0001 C CNN
 	1    7650 2100
@@
 F 0 "R11" H 5970 6146 50  0000 L CNN
 F 1 "100" H 5970 6055 50  0000 L CNN
-F 2 "Resistor_SMD:R_0603_1608Metric" V 5830 6100 50  0001 C CNN
+F 2 "Resistor_SMD:R_0805_2012Metric" V 5830 6100 50  0001 C CNN
 F 3 "~" H 5900 6100 50  0001 C CNN
 	1    5900 6100
@@
 F 0 "R9" H 4970 6146 50  0000 L CNN
 F 1 "100" H 4970 6055 50  0000 L CNN
-F 2 "Resistor_SMD:R_0603_1608Metric" V 4830 6100 50  0001 C CNN
+F 2 "Resistor_SMD:R_0805_2012Metric" V 4830 6100 50  0001 C CNN
 F 3 "~" H 4900 6100 50  0001 C CNN
 	1    4900 6100
@@
 F 0 "R7" H 3970 6146 50  0000 L CNN
 F 1 "100" H 3970 6055 50  0000 L CNN
-F 2 "Resistor_SMD:R_0603_1608Metric" V 3830 6100 50  0001 C CNN
+F 2 "Resistor_SMD:R_0805_2012Metric" V 3830 6100 50  0001 C CNN
 F 3 "~" H 3900 6100 50  0001 C CNN
 	1    3900 6100
@@
 F 0 "R5" H 2970 6146 50  0000 L CNN
 F 1 "100" H 2970 6055 50  0000 L CNN
-F 2 "Resistor_SMD:R_0603_1608Metric" V 2830 6100 50  0001 C CNN
+F 2 "Resistor_SMD:R_0805_2012Metric" V 2830 6100 50  0001 C CNN
 F 3 "~" H 2900 6100 50  0001 C CNN
 	1    2900 6100
@@
 F 0 "R3" H 1970 6146 50  0000 L CNN
 F 1 "100" H 1970 6055 50  0000 L CNN
-F 2 "Resistor_SMD:R_0603_1608Metric" V 1830 6100 50  0001 C CNN
+F 2 "Resistor_SMD:R_0805_2012Metric" V 1830 6100 50  0001 C CNN
 F 3 "~" H 1900 6100 50  0001 C CNN
 	1    1900 6100
@@
 F 0 "R1" H 970 6146 50  0000 L CNN
 F 1 "100" H 970 6055 50  0000 L CNN
-F 2 "Resistor_SMD:R_0603_1608Metric" V 830 6100 50  0001 C CNN
+F 2 "Resistor_SMD:R_0805_2012Metric" V 830 6100 50  0001 C CNN
 F 3 "~" H 900 6100 50  0001 C CNN
 	1    900  6100
@@
 F 0 "R14" H 4550 3200 50  0000 L CNN
 F 1 "10K" H 4550 3100 50  0000 L CNN
-F 2 "Resistor_SMD:R_0603_1608Metric" V 4430 3150 50  0001 C CNN
+F 2 "Resistor_SMD:R_0805_2012Metric" V 4430 3150 50  0001 C CNN
 F 3 "~" H 4500 3150 50  0001 C CNN
 	1    4500 3150
@@
 F 0 "R15" H 4800 3200 50  0000 L CNN
 F 1 "10K" H 4800 3100 50  0000 L CNN
-F 2 "Resistor_SMD:R_0603_1608Metric" V 4680 3150 50  0001 C CNN
+F 2 "Resistor_SMD:R_0805_2012Metric" V 4680 3150 50  0001 C CNN
 F 3 "~" H 4750 3150 50  0001 C CNN
 	1    4750 3150
@@
 F 0 "R16" H 5050 3200 50  0000 L CNN
 F 1 "10K" H 5050 3100 50  0000 L CNN
-F 2 "Resistor_SMD:R_0603_1608Metric" V 4930 3150 50  0001 C CNN
+F 2 "Resistor_SMD:R_0805_2012Metric" V 4930 3150 50  0001 C CNN
 F 3 "~" H 5000 3150 50  0001 C CNN
 	1    5000 3150

Commit message: party operation mode
Parts:
- U1: symbol NUCLEO-L432KC:NUCLEO_L432KC -> CAN_Accessories-rescue:NUCLEO_L432KC-NUCLEO-L432KC
- U2: symbol 2021-02-19_16-08-03:MCP2562FD-E_SN -> CAN_Accessories-rescue:MCP2562FD-E_SN-2021-02-19_16-08-03
Changed lines of the file:
@@
 NoConn ~ 4400 2200
 $Comp
-L NUCLEO-L432KC:NUCLEO_L432KC U1
+L CAN_Accessories-rescue:NUCLEO_L432KC-NUCLEO-L432KC U1
 U 1 1 612C180F
 P 3500 1300
@@
 $EndComp
 $Comp
-L 2021-02-19_16-08-03:MCP2562FD-E_SN U2
+L CAN_Accessories-rescue:MCP2562FD-E_SN-2021-02-19_16-08-03 U2
 U 1 1 612D37CA
 P 9050 1600
